File: LED20RingTiny.sch (KiCad schematic (older format))
At the start: 23 parts, among them IC1 ATTINY45-P, SW1 SW_Push

Commit message: Align LEDs on 5mils grid
Parts:
- IC1: footprint Housings_DIP:DIP-8_W7.62mm_LongPads -> Housings_SOIC:SOIJ-8_5.3x5.3mm_Pitch1.27mm
Changed lines of the file:
@@
 F 0 "IC1" H 6350 4350 50  0000 C CNN
 F 1 "ATTINY45-P" H 8500 3550 50  0000 C CNN
-F 2 "Housings_DIP:DIP-8_W7.62mm_LongPads" H 8500 3950 50  0001 C CIN
+F 2 "Housings_SOIC:SOIJ-8_5.3x5.3mm_Pitch1.27mm" H 8500 3950 50  0001 C CIN
 F 3 "" H 7500 3950 50  0000 C CNN
 	1    7500 3950

Commit message: Improve
Parts:
- added BT1: Battery_Cell, Connectors:CR2032V, symbol Battery_Cell
- SW1: footprint Buttons_Switches_THT:SW_PUSH_6mm -> Buttons_Switches_SMD:SW_SPST_KMR2
Connections:
- net +3V3: now also BT1.1 (+)
- net GND: now also BT1.2 (-)
Changed lines of the file:
@@
 Connection ~ 5700 1650
 Wire Wire Line
-	9150 4600 9150 4050
+	9150 4050 9150 4600
 Wire Wire Line
 	9150 3850 9150 3700
 Wire Wire Line
-	9150 3700 8850 3700
+	8850 3700 9500 3700
 $Comp
 L SW_Push SW1
@@
 F 0 "SW1" H 7400 4650 50  0000 L CNN
 F 1 "SW_Push" H 7350 4490 50  0001 C CNN
-F 2 "Buttons_Switches_THT:SW_PUSH_6mm" H 7350 4750 50  0001 C CNN
+F 2 "Buttons_Switches_SMD:SW_SPST_KMR2" H 7350 4750 50  0001 C CNN
 F 3 "" H 7350 4750 50  0000 C CNN
 	1    7350 4550
@@
 	7550 4550 9150 4550
 Connection ~ 9150 4550
+Connection ~ 9150 4200
+Connection ~ 9150 3700
+$Comp
+L Battery_Cell BT1
+U 1 1 58DE28DD
+P 9500 4000
+F 0 "BT1" H 9600 4100 50  0000 L CNN
+F 1 "Battery_Cell" H 9600 4000 50  0000 L CNN
+F 2 "Connectors:CR2032V" V 9500 4060 50  0001 C CNN
+F 3 "" V 9500 4060 50  0000 C CNN
+	1    9500 4000
+	1    0    0    -1
+$EndComp
 Wire Wire Line
-	8850 4200 9150 4200
-Connection ~ 9150 4200
+	8850 4200 9500 4200
+Wire Wire Line
+	9500 4200 9500 4100
+Wire Wire Line
+	9500 3700 9500 3800
 $EndSCHEMATC
